File: Esquematico_Arm.kicad_sch (KiCad schematic)
At the start: 30 parts, among them J1 Batterry, J10 Servo Motor 5, J2 Motor DC, J3 NEMA17, J4 Resistive Sensor Upper, J5 Touch Sensor Lower, J6 Servo Motor 1, J7 Servo Motor 2, J8 Servo Motor 3, J9 Servo Motor 4, U1 Mini_Ponte_H_L298N, U2 A4988_STEPPER_MOTOR_DRIVER_CA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, U3 CN4015-1, U4 Driver_Conversor3_3_5, U5 ESP32-DEVKIT-V1, U6 Driver_Conversor3_3_5

Commit message: feat(.kicad_sch): att project
Parts:
- added 100nF1, 100nF2: C_Small, Capacitor_THT:C_Disc_D5.1mm_W3.2mm_P5.00mm, symbol Device:C_Small
- added 10uF2, 10uF3: C_Polarized_Small, Capacitor_THT:CP_Radial_D8.0mm_P2.50mm, symbol Device:C_Polarized_Small
- added U1: Driver_Conversor3_3_5, Ponte_H:Conversor_Nivel_Logico, symbol New_Library:Driver_Conversor3_3_5
- added U5: LM2596, symbol Regulador_Tensao:CN4015-1
- U3: renamed from U2; footprint Ponte_H:Driver_A4988 -> MODULE_A4988_STEPPER_MOTOR_DRIVER_CARRIER
- U7: renamed from U5; footprint Ponte_H:ESP32_DEV -> MODULE_ESP32_DEVKIT_V1
- renumbered 100nF1 to 100nF3, 100nF2 to 100nF4, 100nF3 to 100nF5, 100nF4 to 100nF6, 100nF5 to 100nF7, 10uF2 to 10uF4, 10uF3 to 10uF5, 10uF4 to 10uF6, 10uF5 to 10uF7, 10uF6 to 10uF8, U1 to U2, U3 to U4, U4 to U6, U6 to U8
Connections:
- net +12V: now also 100nF1.1, 10uF2.1, U5.1 (Vin)
- net +3.3V: now also U1.3 (LV)
- net +5V: now also U1.10 (HV); no longer U7.30 (VIN)
- net DIR_NEMA_17: now also U1.2 (LV2); no longer U3.8 (DIR)
- net Earth: now also 100nF1.2, 100nF2.2, 10uF2.2, 10uF3.2, U1.4 (GND), U1.9 (GND), U5.2 (GND), U5.4 (GND)
- net IN_1_MOTOR_DC: now also U7.12 (D32), U8.2 (LV2); no longer U2.3 (IN1), U7.11 (D35)
- net IN_2_MOTOR_DC: now also U7.13 (D33), U8.5 (LV3); no longer U2.4 (IN2), U7.12 (D32)
- net Lower_Rotarion_Limit: now also U7.11 (D35); no longer U7.10 (D34)
- net STEP_NEMA_17: now also U1.1 (LV1); no longer U3.7 (STEP)
- net Servo_Motor_4: now also U6.6 (LV4); no longer U8.1 (LV1)
- net Servo_Motor_5: now also U8.1 (LV1); no longer U8.2 (LV2)
- net Servo_Motor_H_4: now also U6.7 (HV4); no longer U8.12 (HV1)
- net Servo_Motor_H_5: now also U8.12 (HV1); no longer U8.11 (HV2)
- net Upper_Rotation_Limit: now also U7.10 (D34); no longer U7.8 (D39)
- net IN_2_MOTOR_DC_H: now reaches U8.8 (HV3)
- net IN_2_MOTOR_DC_H: now also U2.4 (IN2)
- new net +5VD: 100nF2.1, 10uF3.1, U5.3 (Vout), U7.30 (VIN)
- new net DIR_NEMA_17_H: U1.11 (HV2), U3.8 (DIR)
- new net IN_1_MOTOR_DC_H: U2.3 (IN1), U8.11 (HV2)
- new net STEP_NEMA_17_H: U1.12 (HV1), U3.7 (STEP)
- no-connect marks 27 -> 29
Other:
- note removed: "Motor DC - Stall Current: 1A - Rated Current: 0.07A - Stall Torque: 16 kg.cm"
- note removed: "Motor de Passo - Phase Current: 1.5 A"
- note removed: "Servo Motor - Stall Current 2.5 A - Running Current 500-900mA - Stall torque: 11 kgf·cm"
- moved on the sheet: 100uF1, 10uF1, J1, J3, U3, U4, U7

Commit message: feat(.kicad_sch): att pinout
Parts:
- added J?: Base_Pot, TerminalBlock:TerminalBlock_bornier-3_P5.08mm, symbol Connector:Screw_Terminal_01x03
Connections:
- net DIR_NEMA_17: now also U7.15 (D26); no longer U7.18 (D12)
- net STEP_NEMA_17: now also U7.14 (D25); no longer U7.17 (D14)
- no-connect marks 29 -> 27
Other:
- moved on the sheet: 100uF1, 10uF1, J3, U1, U3

Commit message: feat(Arm): Update 12V connector for step motor
Parts:
- added J?: Power_Nema_17, symbol Connector:Screw_Terminal_01x01
- gave numbers to parts that had none: 1
- renumbered J9 to J10, J10 to J11, J6 to J7, J7 to J8, J8 to J9
Connections:
- net +12V: now also J?.1 (Pin_1)
- net +3.3V: now also J6.1 (Pin_1)
- net Earth: now also J6.3 (Pin_3)
- net POTENTIOMETER_BASE: now reaches J6.2 (Pin_2)
- net POTENTIOMETER_BASE: now also U7.16 (D27)
- no-connect marks 27 -> 28
Other:
- moved on the sheet: J3, J6

Commit message: feat(sch): att libraries
Parts:
- removed U1, U6, U8: Driver_Conversor3_3_5, Ponte_H:Conversor_Nivel_Logico, symbol New_Library:Driver_Conversor3_3_5
- removed U2: Mini_Ponte_H_L298N, Ponte_H:Ponte_H, symbol New_Library:Mini_Ponte_H_L298N
- removed U7: ESP32-DEVKIT-V1, MODULE_ESP32_DEVKIT_V1, symbol ESP32-DEVKIT-V1:ESP32-DEVKIT-V1
- added U1, U6, U8: Driver_Conversor3_3_5_1, Ponte_H:Conversor_Nivel_Logico, symbol driver_conversor3_3_5_1:Driver_Conversor3_3_5_1
- added U2: Mini_Ponte_H_L298N, Ponte_H:Ponte_H, symbol mini_ponte_h_l298n:Mini_Ponte_H_L298N
- added U7: ESP32-DEVKIT-V1, Ponte_H:ESP32_DEV, symbol esp32-devkit-v1:ESP32-DEVKIT-V1
- J4: renamed from J?; footprint (none) -> Connector_Pin:Pin_D1.3mm_L11.0mm
- U3: footprint MODULE_A4988_STEPPER_MOTOR_DRIVER_CARRIER -> Ponte_H:Driver_A4988
- U5: footprint (none) -> Ponte_H:Regulador_Tensao
- renumbered J9 to J10, J10 to J11, J11 to J12, J4 to J5, J5 to J6, J6 to J7, J7 to J8, J8 to J9
Connections:
- net +3.3V: now also U1.3 (LV), U6.3 (LV), U7.1 (3V3), U8.3 (LV)
- net +5V: now also U1.10 (HV), U2.1 (Vin), U6.10 (HV), U8.10 (HV)
- net +5VD: now also U7.30 (VIN)
- net DIR_NEMA_17: now also U1.2 (LV2), U7.15 (D26)
- net DIR_NEMA_17_H: now also U1.11 (HV2)
- net Earth: now also U1.4 (GND), U1.9 (GND), U2.2 (GND), U6.4 (GND), U6.9 (GND), U7.2 (GND), U8.4 (GND), U8.9 (GND)
- net IN_1_MOTOR_DC: now also U7.12 (D32), U8.2 (LV2)
- net IN_1_MOTOR_DC_H: now also U2.3 (IN1), U8.11 (HV2)
- net IN_2_MOTOR_DC: now also U7.13 (D33), U8.5 (LV3)
- net IN_2_MOTOR_DC_H: now also U2.4 (IN2), U8.8 (HV3)
- net Lower_Rotarion_Limit: now also U7.11 (D35)
- net POTENTIOMETER_BASE: now also U7.16 (D27)
- net STEP_NEMA_17: now also U1.1 (LV1), U7.14 (D25)
- net STEP_NEMA_17_H: now also U1.12 (HV1)
- net Servo_Motor_1: now also U6.1 (LV1), U7.35 (D18)
- net Servo_Motor_2: now also U6.2 (LV2), U7.38 (D19)
- net Servo_Motor_3: now also U6.5 (LV3), U7.42 (D21)
- net Servo_Motor_4: now also U6.6 (LV4), U7.39 (D22)
- net Servo_Motor_5: now also U7.36 (D23), U8.1 (LV1)
- net Servo_Motor_H_1: now also U6.12 (HV1)
- net Servo_Motor_H_2: now also U6.11 (HV2)
- net Servo_Motor_H_3: now also U6.8 (HV3)
- net Servo_Motor_H_4: now also U6.7 (HV4)
- net Servo_Motor_H_5: now also U8.12 (HV1)
- net Upper_Rotation_Limit: now also U7.10 (D34)
- net at J2.1 (Pin_1): now also U2.8 (Dir_M1)
- net at J2.2 (Pin_2): now also U2.9 (Esq_M1)
